File: CommisDesPintes/CommisDesPintes.sch (KiCad schematic (older format))
At the start: 13 parts

Commit message: Update Schematic
Parts:
- removed D? (x2): D, symbol Device:D
- removed R? (x2): R, symbol Device:R
- added J?: Conn_01x03, symbol Connector_Generic:Conn_01x03
- added QN?: MOSFET_Pair_PN, symbol custom_components:MOSFET_Pair_PN
Connections:
- net GND: now also QN?.1 (S1), QN?.5 (D2), QN?.6 (D2)
- net M_Out: now also U?.4 (R); no longer U?.10 (R)
- net Out: now also U?.5 (Q), QN?.2 (G1), QN?.4 (G2); no longer U?.9 (Q)
- net at C?.2, R?.2: now also U?.2 (THR), U?.6 (TR); no longer U?.12 (THR), U?.8 (TR)
- net at R?.1, R?.1: now also U?.1 (DIS); no longer U?.13 (DIS)
- new net: J?.2 (Pin_2), QN?.3 (S2)
- new net: J?.1 (Pin_1), QN?.7 (D1), QN?.8 (D1)
- new net +12V: J?.3 (Pin_3)
Changed lines of the file:
@@
 $EndDescr
-$Comp
-L Device:R R?
-U 1 1 5E74DF30
-P 6850 1700
-F 0 "R?" V 6643 1700 50  0000 C CNN
-F 1 "R" V 6734 1700 50  0000 C CNN
-F 2 "" V 6780 1700 50  0001 C CNN
-F 3 "~" H 6850 1700 50  0001 C CNN
-	1    6850 1700
-	0    1    1    0
-$EndComp
-$Comp
-L Device:R R?
-U 1 1 5E74E928
-P 6850 2050
-F 0 "R?" V 6643 2050 50  0000 C CNN
-F 1 "R" V 6734 2050 50  0000 C CNN
-F 2 "" V 6780 2050 50  0001 C CNN
-F 3 "~" H 6850 2050 50  0001 C CNN
-	1    6850 2050
-	0    1    1    0
-$EndComp
-$Comp
-L Device:D D?
-U 1 1 5E74F4B2
-P 7150 1700
-F 0 "D?" H 7150 1484 50  0000 C CNN
-F 1 "D" H 7150 1575 50  0000 C CNN
-F 2 "" H 7150 1700 50  0001 C CNN
-F 3 "~" H 7150 1700 50  0001 C CNN
-	1    7150 1700
-	-1   0    0    1
-$EndComp
-$Comp
-L Device:D D?
-U 1 1 5E7503BC
-P 7150 2050
-F 0 "D?" H 7150 1834 50  0000 C CNN
-F 1 "D" H 7150 1925 50  0000 C CNN
-F 2 "" H 7150 2050 50  0001 C CNN
-F 3 "~" H 7150 2050 50  0001 C CNN
-	1    7150 2050
-	-1   0    0    1
-$EndComp
 $Comp
 L power:GND #PWR?
@@
 F 3 "http://www.ti.com/lit/ds/symlink/lm556.pdf" H 4250 2150 50  0001 C CNN
 	1    4250 2150
-	1    0    0    -1
-$EndComp
-$Comp
-L custom_components:LM556 U?
-U 2 1 5E7746EE
-P 4250 3850
-F 0 "U?" H 4550 3450 50  0000 C CNN
-F 1 "LM556" H 4000 4200 50  0000 C CNN
-F 2 "" H 4250 3850 50  0001 C CNN
-F 3 "http://www.ti.com/lit/ds/symlink/lm556.pdf" H 4250 3850 50  0001 C CNN
-	2    4250 3850
 	1    0    0    -1
 $EndComp
@@
 Wire Notes Line
 	2900 3050 5150 3050
+$Comp
+L custom_components:LM556 U?
+U 1 1 5E7746EE
+P 4250 3850
+F 0 "U?" H 4550 3450 50  0000 C CNN
+F 1 "LM556" H 4000 4200 50  0000 C CNN
+F 2 "" H 4250 3850 50  0001 C CNN
+F 3 "http://www.ti.com/lit/ds/symlink/lm556.pdf" H 4250 3850 50  0001 C CNN
+	1    4250 3850
+	1    0    0    -1
+$EndComp
+$Comp
+L custom_components:MOSFET_Pair_PN QN?
+U 1 1 5E7E8347
+P 6650 3050
+F 0 "QN?" H 6650 3715 50  0000 C CNN
+F 1 "MOSFET_Pair_PN" H 6650 3624 50  0000 C CNN
+F 2 "" H 6800 3400 50  0001 C CNN
+F 3 "" H 6800 3400 50  0001 C CNN
+	1    6650 3050
+	1    0    0    -1
+$EndComp
+Wire Wire Line
+	6300 2800 6200 2800
+Wire Wire Line
+	6200 2800 6200 3150
+Wire Wire Line
+	6200 3150 6300 3150
+Wire Wire Line
+	7000 2800 7050 2800
+Wire Wire Line
+	7050 2800 7050 2650
+Wire Wire Line
+	7050 2650 7000 2650
+Wire Wire Line
+	7050 2650 7300 2650
+Connection ~ 7050 2650
+Wire Wire Line
+	6200 2800 6050 2800
+Connection ~ 6200 2800
+$Comp
+L power:GND #PWR?
+U 1 1 5E7F86BA
+P 5850 2900
+F 0 "#PWR?" H 5850 2650 50  0001 C CNN
+F 1 "GND" H 5855 2727 50  0000 C CNN
+F 2 "" H 5850 2900 50  0001 C CNN
+F 3 "" H 5850 2900 50  0001 C CNN
+	1    5850 2900
+	1    0    0    -1
+$EndComp
+Text Label 6050 2800 0    50   ~ 0
+Out
+$Comp
+L power:+12V #PWR?
+U 1 1 5E7FA31B
+P 7700 2550
+F 0 "#PWR?" H 7700 2400 50  0001 C CNN
+F 1 "+12V" H 7715 2723 50  0000 C CNN
+F 2 "" H 7700 2550 50  0001 C CNN
+F 3 "" H 7700 2550 50  0001 C CNN
+	1    7700 2550
+	1    0    0    -1
+$EndComp
+Wire Wire Line
+	7000 3150 7050 3150
+Wire Wire Line
+	7050 3150 7050 3000
+Wire Wire Line
+	7050 3000 7000 3000
+$Comp
+L power:GND #PWR?
+U 1 1 5E80069B
+P 7050 3250
+F 0 "#PWR?" H 7050 3000 50  0001 C CNN
+F 1 "GND" H 7055 3077 50  0000 C CNN
+F 2 "" H 7050 3250 50  0001 C CNN
+F 3 "" H 7050 3250 50  0001 C CNN
+	1    7050 3250
+	1    0    0    -1
+$EndComp
+Wire Wire Line
+	7050 3150 7050 3250
+Connection ~ 7050 3150
+Wire Wire Line
+	5850 2650 5850 2900
+Wire Wire Line
+	5850 2650 6300 2650
+Wire Wire Line
+	6300 3000 6100 3000
+Wire Wire Line
+	6100 3000 6100 3500
+$Comp
+L Connector_Generic:Conn_01x03 J?
+U 1 1 5E8090C8
+P 7400 2350
+F 0 "J?" V 7500 2500 50  0000 R CNN
+F 1 "Conn_01x03" V 7500 2350 50  0000 R CNN
+F 2 "" H 7400 2350 50  0001 C CNN
+F 3 "~" H 7400 2350 50  0001 C CNN
+	1    7400 2350
+	0    -1   -1   0
+$EndComp
+Wire Wire Line
+	7500 2550 7500 2600
+Wire Wire Line
+	7500 2600 7700 2600
+Wire Wire Line
+	7700 2600 7700 2550
+Wire Wire Line
+	6100 3500 7400 3500
+Wire Wire Line
+	7300 2550 7300 2650
+Wire Wire Line
+	7400 3500 7400 2550
 $EndSCHEMATC

Commit message: Update Schematic
Other:
- note added: "IRF7309PbF"
Changed lines of the file:
@@
 Wire Wire Line
 	7400 3500 7400 2550
+Text Notes 6400 3400 0    50   ~ 0
+IRF7309PbF
 $EndSCHEMATC

Commit message: Finished Schematic
Parts:
- removed J?: Conn_01x03, symbol Connector_Generic:Conn_01x03
- removed QN?: MOSFET_Pair_PN, symbol custom_components:MOSFET_Pair_PN
- added C?: 47nF, symbol Device:C
- added C?: 470nF, symbol Device:C
- added C?: 10nF, symbol Device:C
- added C? (x2): 22uF, symbol Device:C
- added C? (x2): 0.1uF, symbol Device:C
- added D?: SS310, symbol Device:D_Schottky
- added J? (x3): Conn_01x02, symbol Connector_Generic:Conn_01x02
- added L?: 22uH, symbol Device:L
- added Q?: FS8205, symbol custom_components:FS8205
- added R?: 7.5kR, symbol Device:R
- added R? (x2): 1kR, symbol Device:R
- added R?: 100R, symbol Device:R
- added SW?: SW_SPDT, symbol Switch:SW_SPDT
- added SW?: SW_SPST, symbol Switch:SW_SPST
- added U?: MAX256, symbol custom_components:MAX256
- added U?: MT3608, symbol custom_components:MT3608
- added U?: FS312F-G, symbol custom_components:FS312F-G
- C?: value 4.7uF -> 2.2uF
Connections:
- net GND: now also C?.1, C?.1, C?.1, C?.1, C?.1, C?.1, J?.1 (Pin_1), Q?.3 (S2), R?.1, R?.2, U?.2 (GND), U?.4 (MODE), U?.6 (GND), U?.7 (GND)
- net Out: now also U?.1 (CK_RS)
- net VCC: now also C?.2, C?.2, C?.2, C?.2, D?.1 (K), R?.1, U?.2 (VCC), U?.3 (VCC)
- net C_F_SEL: now reaches R?.2, U?.2 (THR), U?.6 (TR)
- net C_F_SEL: now also SW?.2 (B); no longer C?.2
- new net: C?.2, SW?.1 (A)
- new net: C?.2, SW?.3 (C)
- new net: J?.2 (Pin_2), U?.5 (ST2)
- new net: J?.1 (Pin_1), U?.8 (ST1)
- new net: C?.2, J?.1 (Pin_1), Q?.1 (S1), U?.6 (GND)
- new net: J?.2 (Pin_2), J?.2 (Pin_2), R?.2, SW?.1 (A)
- new net: D?.2 (A), L?.2, U?.1 (SW)
- new net: R?.1, R?.2, U?.3 (FB)
- new net: Q?.6 (G1), U?.1 (OD)
- new net: R?.2, U?.2 (CS)
- new net: Q?.4 (G2), U?.3 (OC)
- new net: C?.1, R?.1, U?.5 (VCC)
- new net +BATT: C?.2, L?.1, SW?.2 (B), U?.4 (EN), U?.5 (Vin)
- no-connect marks 1 -> 5
Other:
- note added: "BAT"
- note added: "Battery Management System"
- note added: "Boost Converter"
- note added: "CHARGER"
- note added: "H-Bridge"
- note added: "Mode Selection"
- note removed: "IRF7309PbF"
- moved on the sheet: C?, R?, SW?, U?A

Commit message: Annotated components
Parts:
- gave numbers to parts that had none: 30
Connections:
- net C_F_SEL: now also U3.12 (THR), U3.8 (TR); no longer U3.2 (THR), U3.6 (TR)
- net M_Out: now also U3.10 (R); no longer U3.4 (R)
- net Out: now also U3.9 (Q); no longer U3.5 (Q)
- net at R5.1, R6.1: now also U3.13 (DIS); no longer U3.1 (DIS)
